File: RP2040-Breadstick/RP2040-Breadstick.kicad_pcb (KiCad board)
At the start: 6 copper layers, 10.2 x 163.8 mm, 58 parts, among them IC501 LM66200DRLR, J111 Conn_01x01, J112 Conn_01x01, J113 Conn_01x01, J114 Conn_01x01, J115 Conn_01x01, J116 Conn_01x01, J117 Conn_01x01, J118 Conn_01x01, J119 Conn_01x01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

Commit message: Raspberry Breadstick Lite modifications complete.
Parts:
- removed R208, R209: 1k 0603, Resistor_SMD:R_0603_1608Metric
- added ?: , clipboard:a90286b4-b738-4e00-aca9-2c8c50e98d30, F.Cu at (83.6, 148.3)
- added REF**: Breadstick B Silk 5mm, Footprints:Breadstick B Silk 5mm, F.Cu at (86.4, 99.1)
Routing:
- net /RP2040/I2C0-SDA: track 9.74 -> 0.00 mm
- net /RP2040/I2C0-SCL: track 9.73 -> 0.00 mm
- net /3V3: track 57.7 -> 55.7 mm, vias 11 -> 9
- net GND: vias 25 -> 33
Other:
- board text added: "Lite"
- board text added: "Raspberry Breadstick Lite"
- board text added: "locked"
- board text removed: "I"
- board text removed: "Raspberry Breadstick"
- board text removed: "♥"
