File: RP2040-Breadstick/RP2040.kicad_sch (KiCad schematic)
At the start: 20 parts, among them U201 RP2040, U202 16MB Flash, Y201 12MHz

Commit message: Raspberry Breadstick Lite modifications complete.
Parts:
- removed R208, R209: 1k 0603, Resistor_SMD:R_0603_1608Metric, symbol Device:R
Connections:
- net IMU_SCL renamed I2C0-SCL
- net IMU_SDA renamed I2C0-SDA
Changed lines of the file:
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@@
   (junction (at 85.09 97.79) (diameter 0) (color 0 0 0 0)
   )
-  (junction (at 231.14 67.31) (diameter 0) (color 0 0 0 0)
-  )
   (junction (at 91.44 104.14) (diameter 0) (color 0 0 0 0)
   )
@@
   (junction (at 198.12 38.1) (diameter 0) (color 0 0 0 0)
   )
-  (junction (at 238.76 86.36) (diameter 0) (color 0 0 0 0)
-  )
   (junction (at 46.99 152.4) (diameter 0) (color 0 0 0 0)
   )
   (junction (at 142.24 78.74) (diameter 0) (color 0 0 0 0)
-  )
-  (junction (at 231.14 83.82) (diameter 0) (color 0 0 0 0)
   )
   (junction (at 121.92 38.1) (diameter 0) (color 0 0 0 0)
@@
     (stroke (width 0) (type default))
   )
-  (wire (pts (xy 231.14 81.28) (xy 231.14 83.82))
-    (stroke (width 0) (type default))
-  )
   (wire (pts (xy 45.72 106.68) (xy 46.99 106.68))
     (stroke (width 0) (type default))
@@
     (stroke (width 0) (type default))
   )
-  (wire (pts (xy 238.76 67.31) (xy 231.14 67.31))
-    (stroke (width 0) (type default))
-  )
   (wire (pts (xy 46.99 119.38) (xy 46.99 121.92))
     (stroke (width 0) (type default))
@@
     (stroke (width 0) (type default))
   )
-  (wire (pts (xy 238.76 73.66) (xy 238.76 67.31))
-    (stroke (width 0) (type default))
-  )
   (wire (pts (xy 72.39 133.35) (xy 72.39 129.54))
     (stroke (width 0) (type default))
@@
     (stroke (width 0) (type default))
   )
-  (wire (pts (xy 238.76 86.36) (xy 242.57 86.36))
-    (stroke (width 0) (type default))
-  )
-  (wire (pts (xy 193.04 83.82) (xy 231.14 83.82))
+  (wire (pts (xy 193.04 83.82) (xy 215.9 83.82))
     (stroke (width 0) (type default))
   )
@@
     (stroke (width 0) (type default))
   )
-  (wire (pts (xy 193.04 86.36) (xy 238.76 86.36))
-    (stroke (width 0) (type default))
-  )
   (wire (pts (xy 104.14 129.54) (xy 105.41 129.54))
     (stroke (width 0) (type default))
@@
     (stroke (width 0) (type default))
   )
-  (wire (pts (xy 238.76 81.28) (xy 238.76 86.36))
-    (stroke (width 0) (type default))
-  )
   (wire (pts (xy 72.39 139.7) (xy 72.39 143.51))
     (stroke (width 0) (type default))
@@
     (stroke (width 0) (type default))
   )
-  (wire (pts (xy 231.14 62.23) (xy 231.14 67.31))
-    (stroke (width 0) (type default))
-  )
   (wire (pts (xy 121.92 30.48) (xy 113.03 30.48))
     (stroke (width 0) (type default))
@@
     (stroke (width 0) (type default))
   )
-  (wire (pts (xy 231.14 83.82) (xy 242.57 83.82))
-    (stroke (width 0) (type default))
-  )
   (wire (pts (xy 46.99 118.11) (xy 46.99 119.38))
     (stroke (width 0) (type default))
@@
     (stroke (width 0) (type default))
   )
-  (wire (pts (xy 231.14 67.31) (xy 231.14 73.66))
-    (stroke (width 0) (type default))
-  )
   (wire (pts (xy 121.92 38.1) (xy 121.92 30.48))
     (stroke (width 0) (type default))
   )
   (wire (pts (xy 121.92 40.64) (xy 147.32 40.64))
+    (stroke (width 0) (type default))
+  )
+  (wire (pts (xy 193.04 86.36) (xy 215.9 86.36))
     (stroke (width 0) (type default))
   )
@@
     (effects (font (size 1.27 1.27)) (justify left bottom))
   )
-  (label "I2C0-SCL" (at 213.36 86.36 0) (fields_autoplaced)
-    (effects (font (size 1.27 1.27)) (justify left bottom))
-  )
-  (label "I2C0-SDA" (at 213.36 83.82 0) (fields_autoplaced)
+  (label "I2C0-SCL" (at 205.74 86.36 0) (fields_autoplaced)
+    (effects (font (size 1.27 1.27)) (justify left bottom))
+  )
+  (label "I2C0-SDA" (at 205.74 83.82 0) (fields_autoplaced)
     (effects (font (size 1.27 1.27)) (justify left bottom))
   )
@@
     (effects (font (size 1.27 1.27)) (justify left))
   )
-  (hierarchical_label "3V3_LDO" (shape input) (at 231.14 62.23 180) (fields_autoplaced)
-    (effects (font (size 1.27 1.27)) (justify right))
-  )
   (hierarchical_label "~{RESET}" (shape input) (at 45.72 87.63 180) (fields_autoplaced)
     (effects (font (size 1.27 1.27)) (justify right))
@@
   )
   (hierarchical_label "D13" (shape tri_state) (at 196.85 106.68 0) (fields_autoplaced)
-    (effects (font (size 1.27 1.27)) (justify left))
-  )
-  (hierarchical_label "IMU_SCL" (shape output) (at 242.57 86.36 0) (fields_autoplaced)
-    (effects (font (size 1.27 1.27)) (justify left))
-  )
-  (hierarchical_label "IMU_SDA" (shape bidirectional) (at 242.57 83.82 0) (fields_autoplaced)
     (effects (font (size 1.27 1.27)) (justify left))
   )
@@
     )
   )
-  (symbol (lib_id "Device:R") (at 238.76 77.47 0) (mirror x) (unit 1)
-    (in_bom yes) (on_board yes) (dnp no)
-    (property "Reference" "R209" (at 234.315 78.105 90)
-      (effects (font (size 1.27 1.27)) (justify left))
-    )
-    (property "Value" "1k 0603" (at 236.22 72.39 90)
-      (effects (font (size 1.27 1.27)) (justify left))
-    )
-    (property "Footprint" "Resistor_SMD:R_0603_1608Metric" (at 236.982 77.47 90)
-      (effects (font (size 1.27 1.27)) hide)
-    )
-    (property "Datasheet" "~" (at 238.76 77.47 0)
-      (effects (font (size 1.27 1.27)) hide)
-    )
-    (property "JLCPCB P/N" "" (at 238.76 77.47 0)
-      (effects (font (size 1.27 1.27)) hide)
-    )
-    (property "Digikey" "311-1.00KHRCT-ND" (at 238.76 77.47 0)
-      (effects (font (size 1.27 1.27)) hide)
-    )
-    (property "Manufacturer" "YAGEO" (at 238.76 77.47 0)
-      (effects (font (size 1.27 1.27)) hide)
-    )
-    (property "Manufacturer_Part_Number" "RC0603FR-071KL" (at 238.76 77.47 0)
-      (effects (font (size 1.27 1.27)) hide)
-    )
-    (property "Mouser" "603-RC0603FR-071KL" (at 238.76 77.47 0)
-      (effects (font (size 1.27 1.27)) hide)
-    )
-    (property "Package" "0603" (at 238.76 77.47 0)
-      (effects (font (size 1.27 1.27)) hide)
-    )
-    (property "LCSC" "" (at 238.76 77.47 0)
-      (effects (font (size 1.27 1.27)) hide)
-    )
-    (pin "1")
-    (pin "2")
-    (instances
-      (project "RP2040-Breadstick"
-        (path "/c1b11207-7c0a-49b3-a41d-2fe677d5f3b8/3e7bcc2a-10c2-45cd-9897-4c0007e1c7fc"
-          (reference "R209") (unit 1)
-        )
-      )
-    )
-  )
   (symbol (lib_id "power:GND") (at 113.03 45.72 0) (unit 1)
     (in_bom yes) (on_board yes) (dnp no) (fields_autoplaced)
@@
         )
       )
-    )
-  )
-  (symbol (lib_id "Device:R") (at 231.14 77.47 0) (mirror x) (unit 1)
-    (in_bom yes) (on_board yes) (dnp no)
-    (property "Reference" "R208" (at 226.695 78.105 90)
-      (effects (font (size 1.27 1.27)) (justify left))
-    )
-    (property "Value" "1k 0603" (at 228.6 72.39 90)
-      (effects (font (size 1.27 1.27)) (justify left))
-    )
-    (property "Footprint" "Resistor_SMD:R_0603_1608Metric" (at 229.362 77.47 90)
-      (effects (font (size 1.27 1.27)) hide)
-    )
-    (property "Datasheet" "~" (at 231.14 77.47 0)
-      (effects (font (size 1.27 1.27)) hide)
-    )
-    (property "JLCPCB P/N" "" (at 231.14 77.47 0)
-      (effects (font (size 1.27 1.27)) hide)
-    )
-    (property "Digikey" "311-1.00KHRCT-ND" (at 231.14 77.47 0)
-      (effects (font (size 1.27 1.27)) hide)
-    )
-    (property "Manufacturer" "YAGEO" (at 231.14 77.47 0)
-      (effects (font (size 1.27 1.27)) hide)
-    )
-    (property "Manufacturer_Part_Number" "RC0603FR-071KL" (at 231.14 77.47 0)
-      (effects (font (size 1.27 1.27)) hide)
-    )
-    (property "Mouser" "603-RC0603FR-071KL" (at 231.14 77.47 0)
-      (effects (font (size 1.27 1.27)) hide)
-    )
-    (property "Package" "0603" (at 231.14 77.47 0)
-      (effects (font (size 1.27 1.27)) hide)
-    )
-    (property "LCSC" "" (at 231.14 77.47 0)
-      (effects (font (size 1.27 1.27)) hide)
-    )
-    (pin "1")
-    (pin "2")
-    (instances
-      (project "RP2040-Breadstick"
-        (path "/c1b11207-7c0a-49b3-a41d-2fe677d5f3b8/3e7bcc2a-10c2-45cd-9897-4c0007e1c7fc"
-          (reference "R208") (unit 1)
-        )
-      )
